Commit message: Added gripper movement capabilities
Grippers can be actuated in RVIz, still need to figure out how to control it on the real YuMi

File: yumi_description/urdf/yumi_servo_gripper.xacro (robot description, xacro)
@@ -47,5 +47,5 @@
       </collision>
     </link>
-    <joint name="${name}_joint" type="prismatic">
+    <joint name="${name}_joint_r" type="prismatic">
       <parent link="${name}_base"/>
       <child link="${name}_finger_r"/>
@@ -76,5 +76,5 @@
       </collision>
     </link>
-    <joint name="${name}_joint_m" type="prismatic">
+    <joint name="${name}_joint_l" type="prismatic">
       <parent link="${name}_base"/>
       <child link="${name}_finger_l"/>
@@ -83,5 +83,4 @@
       <limit lower="0" upper="0.025" effort="${max_effort}" velocity="0.02" />
       <dynamics damping="${joint_damping}"/>
-      <mimic joint="${name}_joint"/>
     </joint>
     <link name="${name}_finger_l">

Commit message: Modified files for gripper action
Modified relevent files to allow gripper and arm movements. Still needs to be tested.

File: yumi_description/urdf/yumi_servo_gripper.xacro (robot description, xacro)
@@ -83,4 +83,5 @@
       <limit lower="0" upper="0.025" effort="${max_effort}" velocity="0.02" />
       <dynamics damping="${joint_damping}"/>
+      <mimic joint="${name}_joint_r"/>
     </joint>
     <link name="${name}_finger_l">
