Commit message: Added proper VI sensor properties to xacro
Added VI sensor properties to xacro (frames, etc), and updated workspace to include repo containing VI sensor properties xacro file

File: yumi_description/urdf/camera_assembly.xacro (robot description, xacro)
@@ -3,9 +3,10 @@
   PROGRAMMER: Frederick Wachter
   DATE CREATED: 2016-05-30
-  LAST MODIFIED: 2016-05-30
   PURPOSE: Provide colors for the different objects in the YuMi workspace
 -->
 <robot name="yumi" xmlns:xacro="http://www.ros.org/wiki/xacro">
-  <xacro:macro name="camera_assembly" params="parent">
+  <!-- Include VI Sensor Macro -->
+  <xacro:include filename="$(find rotors_description)/urdf/component_snippets.xacro" />
+  <xacro:macro name="camera_assembly" params="parent vi_namespace enable_cameras enable_depth enable_ground_truth">
     <!--                         -->
     <!--     CAMERA ASSEMBLY     -->
@@ -83,4 +84,12 @@
       </collision>
     </link>
+    <xacro:vi_sensor_macro
+      namespace="${vi_namespace}"
+      parent_link="camera_holder"
+      enable_cameras="${enable_cameras}"
+      enable_depth="${enable_depth}"
+      enable_ground_truth="${enable_ground_truth}">
+      <origin xyz="0.0 0.0 0.6" rpy="0 0 0" />
+    </xacro:vi_sensor_macro>
     <joint name="creative_to_holder" type="fixed">
       <parent link="camera_holder"/>
@@ -88,9 +97,4 @@
       <origin rpy="0 0 0" xyz="-0.002 0.0765 0.0335"/>
     </joint>
-    <joint name="vi_to_holder" type="fixed">
-      <parent link="camera_holder"/>
-      <child link="vi_sensor"/>
-      <origin rpy="0 0 0" xyz="0 -0.0138 0.028"/>
-    </joint>
   </xacro:macro>
 </robot>

File: yumi_description/urdf/utilities.xacro (robot description, xacro)
@@ -3,5 +3,4 @@
   PROGRAMMER: Frederick Wachter
   DATE CREATED: 2016-05-30
-  LAST MODIFIED: 2016-05-30
   PURPOSE: Provide constants and modeling macros for YuMi
   REFERENCE: https://github.com/rtkg/yumi
@@ -10,4 +9,5 @@
   <!-- Constants -->
   <xacro:property name="PI" value="3.1415926535897931"/>
+  <xacro:property name="vi_namespace" value="vi_sensor"/>
   <!-- Model Properties -->
   <xacro:property name="hardware_interface" value="yumi"/>

File: yumi_description/urdf/yumi.urdf.xacro (robot description, xacro)
@@ -3,5 +3,4 @@
   PROGRAMMER: Frederick Wachter
   DATE CREATED: 2016-05-30
-  LAST MODIFIED: 2016-05-30
   PURPOSE: Import necessary files to build YuMi URDF with workspace
 -->
@@ -45,4 +44,6 @@
   </xacro:yumi_servo_gripper>
   <!-- Define Macros for Camera Assembly Import -->
-  <xacro:camera_assembly parent="yumi_link_7_l"/>
+  <xacro:camera_assembly parent="yumi_link_7_l" vi_namespace="${vi_namespace}"
+    enable_cameras="$(arg enable_cameras)" enable_depth="$(arg enable_depth)" enable_ground_truth="$(arg enable_ground_truth)"
+  />
 </robot>

Commit message: Updated ROS files for proper condifuration with controller settings
Fixed issues with Gripper commands being sent over to YuMi, still need to add custom controller abilities

File: yumi_description/urdf/camera_assembly.xacro (robot description, xacro)
@@ -8,5 +8,5 @@
   <!-- Include VI Sensor Macro -->
   <xacro:include filename="$(find rotors_description)/urdf/component_snippets.xacro" />
-  <xacro:macro name="camera_assembly" params="parent vi_namespace enable_cameras enable_depth enable_ground_truth">
+  <xacro:macro name="camera_assembly" params="parent vi_namespace enable_cameras enable_depth enable_ground_truth PI">
     <!--                         -->
     <!--     CAMERA ASSEMBLY     -->
@@ -68,20 +68,4 @@
       </collision>
     </link>
-    <link name="vi_sensor">
-      <visual>
-        <origin rpy="0 -1.575 -1.5098" xyz="0 0 0"/>
-        <geometry>
-          <mesh filename="package://yumi_description/meshes/camera/vi_sensor.stl"/>
-        </geometry>
-        <material name="Drexel_Blue"/>
-      </visual>
-      <collision>
-        <origin rpy="0 -1.575 -1.508" xyz="0 0 0"/>
-        <geometry>
-          <mesh filename="package://yumi_description/meshes/camera/vi_sensor.stl"/>
-        </geometry>
-        <material name="Drexel_Blue"/>
-      </collision>
-    </link>
     <xacro:vi_sensor_macro
       namespace="${vi_namespace}"
@@ -90,5 +74,5 @@
       enable_depth="${enable_depth}"
       enable_ground_truth="${enable_ground_truth}">
-      <origin xyz="0.0 0.0 0.6" rpy="0 0 0" />
+      <origin xyz="-0.003 -0.0138 0.02825" rpy="${PI} ${-PI/2 + 0.0063} ${PI/2}" />
     </xacro:vi_sensor_macro>
     <joint name="creative_to_holder" type="fixed">

File: yumi_description/urdf/yumi.urdf.xacro (robot description, xacro)
@@ -4,4 +4,8 @@
   DATE CREATED: 2016-05-30
   PURPOSE: Import necessary files to build YuMi URDF with workspace
+  NECESSARY INPUTS:
+    - enable_cameras: true/false
+    - enable_depth: true/false
+    - enable_ground_truth: true/false
 -->
 <robot name="yumi" xmlns:xacro="http://www.ros.org/wiki/xacro">
@@ -31,4 +35,5 @@
   <!--    MACRO DEFINITIONS    -->
   <!--                  		   -->
+  <!-- Set defaults -->
   <!-- Define Macros for YuMi Import -->
   <xacro:yumi name="yumi" hardware_interface="${hardware_interface}" parent="world">
@@ -44,5 +49,5 @@
   </xacro:yumi_servo_gripper>
   <!-- Define Macros for Camera Assembly Import -->
-  <xacro:camera_assembly parent="yumi_link_7_l" vi_namespace="${vi_namespace}"
+  <xacro:camera_assembly parent="yumi_link_7_l" vi_namespace="${vi_namespace}" PI="${PI}"
     enable_cameras="$(arg enable_cameras)" enable_depth="$(arg enable_depth)" enable_ground_truth="$(arg enable_ground_truth)"
   />

File: yumi_description/urdf/yumi_servo_gripper.xacro (robot description, xacro)
@@ -81,5 +81,5 @@
       <origin xyz="0 0.0065 0.0837" rpy="0 0 ${PI}"/>
       <axis xyz="-1 0 0"/>
-      <limit lower="0" upper="0.025" effort="${max_effort}" velocity="0.02" />
+      <limit lower="0" upper="0.024" effort="${max_effort}" velocity="0.02" />
       <dynamics damping="${joint_damping}"/>
       <mimic joint="${name}_joint_r"/>

Commit message: Changed camera name and updated end-effectors

File: yumi_description/urdf/camera_assembly.xacro (robot description, xacro)
@@ -51,5 +51,5 @@
       </collision>
     </link>
-    <link name="creative_camera">
+    <link name="sr300_sensor">
       <visual>
         <origin rpy="0 0 0" xyz="0 0 0"/>
@@ -85,5 +85,5 @@
     <joint name="creative_to_holder" type="fixed">
       <parent link="camera_holder"/>
-      <child link="creative_camera"/>
+      <child link="sr300_sensor"/>
       <origin rpy="0 0 0" xyz="-0.002 0.0765 0.0335"/>
     </joint>
