Commit message: Modified workspace for new workspace for YuMi

File: yumi_description/urdf/workspace.xacro (robot description, xacro)
@@ -7,5 +7,5 @@
 -->
 <robot name="yumi" xmlns:xacro="http://www.ros.org/wiki/xacro">
-  <xacro:macro name="workspace" params="stand_parent table_parent *origin">
+  <xacro:macro name="workspace" params="stand_parent table_parent">
     <!--                         -->
     <!--          TABLE          -->
@@ -14,16 +14,16 @@
       <parent link="${table_parent}"/>
       <child link="table"/>
-      <insert_block name="origin"/>
+      <origin rpy="0 0 0" xyz="0.334 -0.01 -0.013"/>
     </joint>
     <link name="table"/>
-    <joint name="table_top_to_table" type="fixed">
+    <joint name="table_main_to_table" type="fixed">
       <parent link="table"/>
-      <child link="table_top"/>
+      <child link="table_main"/>
       <origin rpy="0 0 0" xyz="0 0 0"/>
     </joint>
-    <link name="table_top">
+    <link name="table_main">
       <visual>
         <geometry>
-          <box size="0.8 1.6 0.026"/>
+          <box size="1.6 0.8 0.026"/>
         </geometry>
         <origin rpy="0 0 0" xyz="0 0 0"/>
@@ -32,5 +32,26 @@
       <collision>
         <geometry>
-          <box size="0.8 1.6 0.026"/>
+          <box size="1.6 0.8 0.026"/>
+        </geometry>
+        <origin rpy="0 0 0" xyz="0 0 0"/>
+        <material name="Ivory"/>
+      </collision>
+    </link>
+    <joint name="table_two_to_table" type="fixed">
+      <parent link="table"/>
+      <child link="table_two"/>
+      <origin rpy="0 0 0" xyz="-0.4 1.3 0"/>
+    </joint>
+    <link name="table_two">
+      <visual>
+        <geometry>
+          <box size="0.8 1.8 0.026"/>
+        </geometry>
+        <origin rpy="0 0 0" xyz="0 0 0"/>
+        <material name="Ivory"/>
+      </visual>
+      <collision>
+        <geometry>
+          <box size="0.8 1.8 0.026"/>
         </geometry>
         <origin rpy="0 0 0" xyz="0 0 0"/>

File: yumi_description/urdf/yumi.urdf.xacro (robot description, xacro)
@@ -37,7 +37,5 @@
   </xacro:yumi>
   <!-- Define Macros for Workspace Import -->
-  <xacro:workspace stand_parent="yumi_body" table_parent="world">
-    <origin rpy="0 0 0" xyz="-0.07 0.54 -0.013"/>
-  </xacro:workspace>
+  <xacro:workspace stand_parent="yumi_body" table_parent="world"/>
   <!-- Define Macros for Right Servo Gripper Import -->
   <xacro:yumi_servo_gripper name="gripper_r" hardware_interface="${hardware_interface}" parent="yumi_link_7_r">

Commit message: Added table origin in relation to world as parameter to XACRO files
In accordance to comment from pull request

File: yumi_description/urdf/workspace.xacro (robot description, xacro)
@@ -7,5 +7,5 @@
 -->
 <robot name="yumi" xmlns:xacro="http://www.ros.org/wiki/xacro">
-  <xacro:macro name="workspace" params="stand_parent table_parent">
+  <xacro:macro name="workspace" params="stand_parent table_parent *origin">
     <!--                         -->
     <!--          TABLE          -->
@@ -14,5 +14,5 @@
       <parent link="${table_parent}"/>
       <child link="table"/>
-      <origin rpy="0 0 0" xyz="0.334 -0.01 -0.013"/>
+      <insert_block name="origin"/>
     </joint>
     <link name="table"/>

File: yumi_description/urdf/yumi.urdf.xacro (robot description, xacro)
@@ -37,5 +37,7 @@
   </xacro:yumi>
   <!-- Define Macros for Workspace Import -->
-  <xacro:workspace stand_parent="yumi_body" table_parent="world"/>
+  <xacro:workspace stand_parent="yumi_body" table_parent="world">
+    <origin rpy="0 0 0" xyz="0.334 -0.01 -0.013"/>
+  </xacro:workspace>
   <!-- Define Macros for Right Servo Gripper Import -->
   <xacro:yumi_servo_gripper name="gripper_r" hardware_interface="${hardware_interface}" parent="yumi_link_7_r">

Commit message: Added lead-through script, modified XACRO files, adjusted RAPID for lead-through
Lead-through files allows for the arm to be moved to a location and the postion can then be stored by publishing a set of commands. XACRO files were modified to fix the issue of not having a fixed joint. YuMi and workspace is now attached to a link called Workspace. Changed RAPID files in order to allow only the state servers to be run in order to allow for the arms to be put into lead-through mode for the lead-through script.

File: yumi_description/urdf/workspace.xacro (robot description, xacro)
@@ -11,5 +11,5 @@
     <!--          TABLE          -->
     <!--                         -->
-    <joint name="world_to_table" type="fixed">
+    <joint name="${table_parent}_to_table" type="fixed">
       <parent link="${table_parent}"/>
       <child link="table"/>

File: yumi_description/urdf/yumi.urdf.xacro (robot description, xacro)
@@ -30,6 +30,6 @@
   <!--     LINK DEFINITIONS    -->
   <!--                  		   -->
-  <!-- World Fixed Link for YuMi -->
-  <link name="world"/>
+  <!-- Fixed Link for Entire Workspace -->
+  <link name="workspace"/>
   <!--                  		   -->
   <!--    MACRO DEFINITIONS    -->
@@ -37,9 +37,9 @@
   <!-- Set defaults -->
   <!-- Define Macros for YuMi Import -->
-  <xacro:yumi name="yumi" hardware_interface="${hardware_interface}" parent="world">
+  <xacro:yumi name="yumi" hardware_interface="${hardware_interface}" parent="workspace">
 	  <origin xyz="0 0 0.1" rpy="0 0 0"/> <!-- Bring bottom of YuMi to (x,y) plane -->
   </xacro:yumi>
   <!-- Define Macros for Workspace Import -->
-  <xacro:workspace stand_parent="yumi_body" table_parent="world">
+  <xacro:workspace stand_parent="yumi_body" table_parent="workspace">
     <origin rpy="0 0 0" xyz="0.334 -0.01 -0.013"/>
   </xacro:workspace>

Commit message: Finalize base code for lead through and main script. Need to update IK solver when equation for arm angle is found

File: yumi_description/urdf/workspace.xacro (robot description, xacro)
@@ -62,5 +62,5 @@
     <!--       YUMI STAND        -->
     <!--                         -->
-    <joint name="stand_to_world" type="fixed">
+    <joint name="stand_to_yumi" type="fixed">
       <parent link="${stand_parent}"/>
       <child link="stand"/>

File: yumi_description/urdf/yumi.urdf.xacro (robot description, xacro)
@@ -39,9 +39,9 @@
   <!-- Define Macros for YuMi Import -->
   <xacro:yumi name="yumi" hardware_interface="${hardware_interface}" parent="workspace">
-	  <origin xyz="0 0 0.1" rpy="0 0 0"/> <!-- Bring bottom of YuMi to (x,y) plane -->
+	  <origin xyz="0 0 0" rpy="0 0 0"/> <!-- Bring bottom of YuMi to (x,y) plane -->
   </xacro:yumi>
   <!-- Define Macros for Workspace Import -->
   <xacro:workspace stand_parent="yumi_body" table_parent="workspace">
-    <origin rpy="0 0 0" xyz="0.334 -0.01 -0.013"/>
+    <origin rpy="0 0 0" xyz="0.334 -0.01 -0.113"/>
   </xacro:workspace>
   <!-- Define Macros for Right and Left Servo Gripper Import -->

File: yumi_description/urdf/yumi_servo_gripper.xacro (robot description, xacro)
@@ -106,4 +106,11 @@
       </collision>
     </link>
+    <joint name="${name}_tcp" type="fixed">
+      <parent link="${name}_base"/>
+      <child link="${name}_tcp"/>
+      <origin xyz="0 0 0.1337" rpy="0 0 0"/>
+      <axis xyz="0 0 1"/>
+    </joint>
+    <link name="${name}_tcp"/>
     <!--                              -->
     <!--   YuMi Gripper Extensions    -->

Commit message: Finishing up first version of YuMi node. Adjusted TF tree

File: yumi_description/urdf/workspace.xacro (robot description, xacro)
@@ -11,12 +11,6 @@
     <!--          TABLE          -->
     <!--                         -->
-    <joint name="${table_parent}_to_table" type="fixed">
+    <joint name="table_main_to_${table_parent}" type="fixed">
       <parent link="${table_parent}"/>
-      <child link="table"/>
-      <insert_block name="origin"/>
-    </joint>
-    <link name="table"/>
-    <joint name="table_main_to_table" type="fixed">
-      <parent link="table"/>
       <child link="table_main"/>
       <origin rpy="0 0 0" xyz="0 0 0"/>
@@ -38,6 +32,6 @@
       </collision>
     </link>
-    <joint name="table_two_to_table" type="fixed">
-      <parent link="table"/>
+    <joint name="table_two_to_${table_parent}" type="fixed">
+      <parent link="${table_parent}"/>
       <child link="table_two"/>
       <origin rpy="0 0 0" xyz="-0.4 1.3 0"/>
@@ -67,11 +61,5 @@
       <origin rpy="0 0 0" xyz="0 0 0"/>
     </joint>
-    <link name="stand"/>
-    <joint name="base_to_stand" type="fixed">
-      <parent link="stand"/>
-      <child link="stand_base"/>
-      <origin rpy="0 0 0" xyz="0 0 0"/>
-    </joint>
-    <link name="stand_base">
+    <link name="stand">
       <visual>
         <origin rpy="0 0 0" xyz="165.03939 -0.25716 0.00014"/>

File: yumi_description/urdf/yumi.urdf.xacro (robot description, xacro)
@@ -4,5 +4,5 @@
   DATE CREATED: 2016-05-30
   PURPOSE: Import necessary files to build YuMi URDF with workspace
-  NECESSARY INPUTS:
+  NECESSARY INPUTS FOR VI SENSOR:
     - enable_cameras: true/false
     - enable_depth: true/false
@@ -37,13 +37,13 @@
   <!--                  		   -->
   <!-- Set defaults -->
-  <!-- Define Macros for YuMi Import -->
-  <xacro:yumi name="yumi" hardware_interface="${hardware_interface}" parent="workspace">
-	  <origin xyz="0 0 0" rpy="0 0 0"/> <!-- Bring bottom of YuMi to (x,y) plane -->
-  </xacro:yumi>
   <!-- Define Macros for Workspace Import -->
   <xacro:workspace stand_parent="yumi_body" table_parent="workspace">
-    <origin rpy="0 0 0" xyz="0.334 -0.01 -0.113"/>
+    <origin xyz="0.334 -0.01 -0.113" rpy="0 0 0"/>
   </xacro:workspace>
-  <!-- Define Macros for Right and Left Servo Gripper Import -->
+  <!-- Define Macros for YuMi Import -->
+  <xacro:yumi name="yumi" hardware_interface="${hardware_interface}" parent="table_main">
+	  <origin xyz="0 0 0.113" rpy="0 0 0"/> <!-- Bring bottom of YuMi to (x,y) plane -->
+  </xacro:yumi>
+  <!-- Define Macros for Right Servo Gripper Import -->
   <xacro:yumi_servo_gripper name="gripper_r" hardware_interface="${hardware_interface}" parent="yumi_link_7_r">
   	<origin xyz="0 0 0.007" rpy="0 0 ${PI}"/>
@@ -56,4 +56,5 @@
   </xacro:unless>
   <xacro:if value="$(arg two_grippers)">
+    <!-- Define Macros for Left Servo Gripper Import -->
     <xacro:yumi_servo_gripper name="gripper_l" hardware_interface="${hardware_interface}" parent="yumi_link_7_l">
       <origin xyz="0 0 0.007" rpy="0 0 ${PI}"/>

File: yumi_description/urdf/yumi.xacro (robot description, xacro)
@@ -1,8 +1,6 @@
 <?xml version="1.0"?>
 <!--
-  PROGRAMMER: Frederick Wachter
+  MODIFIER: Frederick Wachter - wachterfreddy@gmail.com
   DATE CREATED: 2016-05-30
-  LAST MODIFIED: 2016-05-30
-  PURPOSE: Provide colors for the different objects in the YuMi workspace
   REFERENCE: https://github.com/rtkg/yumi
 -->

Commit message: Final addition to leap interface, adjustment of URDF, added leap commands to setup_ws file

File: yumi_description/urdf/workspace.xacro (robot description, xacro)
@@ -7,5 +7,5 @@
 -->
 <robot name="yumi" xmlns:xacro="http://www.ros.org/wiki/xacro">
-  <xacro:macro name="workspace" params="stand_parent table_parent *origin">
+  <xacro:macro name="workspace" params="stand_parent table_parent">
     <!--                         -->
     <!--          TABLE          -->

File: yumi_description/urdf/yumi.urdf.xacro (robot description, xacro)
@@ -38,10 +38,8 @@
   <!-- Set defaults -->
   <!-- Define Macros for Workspace Import -->
-  <xacro:workspace stand_parent="yumi_body" table_parent="workspace">
-    <origin xyz="0.334 -0.01 -0.113" rpy="0 0 0"/>
-  </xacro:workspace>
+  <xacro:workspace stand_parent="yumi_body" table_parent="workspace"></xacro:workspace>
   <!-- Define Macros for YuMi Import -->
   <xacro:yumi name="yumi" hardware_interface="${hardware_interface}" parent="table_main">
-	  <origin xyz="0 0 0.113" rpy="0 0 0"/> <!-- Bring bottom of YuMi to (x,y) plane -->
+	  <origin xyz="-0.333 0 0.113" rpy="0 0 0"/> <!-- Bring bottom of YuMi to (x,y) plane -->
   </xacro:yumi>
   <!-- Define Macros for Right Servo Gripper Import -->
