Commit message: Basic cartesion waypoint planning working (yumi.xacro changed to start in non-collision state)

File: yumi_description/urdf/yumi.xacro (robot description, xacro)
@@ -45,5 +45,5 @@
       <parent link="${name}_body"/>
       <child link="${name}_link_1_r"/>
-      <origin xyz="0.05355 -0.0725 0.41492" rpy="-0.9795   -0.5682   -2.3155"/>
+      <origin xyz="0.05355 -0.0725 0.41492" rpy="1 0 0"/> <!---0.9795   -0.5682   -2.3155-->
       <axis xyz="0 0 1"/>
       <limit lower="${-168.5 * PI / 180}" upper="${168.5 * PI / 180}"
@@ -150,5 +150,5 @@
       <parent link="${name}_link_3_r"/>
       <child link="${name}_link_4_r"/>
-      <origin xyz="-0.04188 0.0 0.07873" rpy="${PI / 2} ${- PI / 2} 0.0"/>
+      <origin xyz="-0.04188 0.0 0.07873" rpy="${PI / 2} ${ PI / 2} 0"/> <!-- ${PI / 2} ${- PI / 2} 0.0 -->
       <axis xyz="0 0 1"/>
       <limit lower="${-123.5 * PI / 180}" upper="${80 * PI / 180}"
